File: KicadV7/gemma20Pico.kicad_pcb (KiCad board)
At the start: 2 copper layers, 60 x 45 mm, 12 parts, among them J1-Prox1 I2C_CH0, J2-Prox0 I2C_CH1, J3-Motor1 DC-Motor, J4-BAT1 3.7V Battery, J5-Servo1 Servo, J6-Pot1 Pot, J7-Pot2 Pot, U1-RPI-Pico1 Pico

Commit message: Cleanup
Parts:
- added C1: C_Polarized_Small_US, Capacitor_THT:CP_Radial_D5.0mm_P2.50mm, F.Cu at (93.5, 106.0)
Routing:
- net /SCL0: track 20.7 -> 19.3 mm
- net +BATT: track 83.5 -> 82.9 mm, vias 2 -> 1
- net /SDA1: track 18.2 -> 17.7 mm
- net GND: vias 1 -> 10
Other:
- board text added: "PicoRC 1.1 USN 2023"
- board text removed: "PicoRC 1.1 Jan & Rune"
